File: coin_counter/coin_counter/coin_counter.kicad_pcb (KiCad board)
At the start: 2 copper layers, 13 parts, among them J1 Q_EMT, J2 N_EMT, J3 P_EMT, J4 D_EMT, J5 Mom, J6 D_RCV, J7 P_RCV, J8 N_RCV, J9 Q_RCV

Commit message: more
Parts:
- added A1: Arduino_Nano_Every, Module:Arduino_Nano, F.Cu at (180.8, 98.1)
- added J10: Mom, Connector_JST:JST_XH_B6B-XH-A_1x06_P2.50mm_Vertical, F.Cu at (181.0, 75.5)
- added J11: Power, Connector_JST:JST_XH_B2B-XH-A_1x02_P2.50mm_Vertical, F.Cu at (198.0, 83.0)
- added R1: 220 Ohm, Resistor_THT:R_Axial_DIN0204_L3.6mm_D1.6mm_P5.08mm_Vertical, F.Cu at (193.0, 68.5)
- added R2: 220 Ohm, Resistor_THT:R_Axial_DIN0204_L3.6mm_D1.6mm_P5.08mm_Vertical, F.Cu at (190.0, 68.5)
- added R3: 220 Ohm, Resistor_THT:R_Axial_DIN0204_L3.6mm_D1.6mm_P5.08mm_Vertical, F.Cu at (187.0, 68.5)
- added R4: 220 Ohm, Resistor_THT:R_Axial_DIN0204_L3.6mm_D1.6mm_P5.08mm_Vertical, F.Cu at (184.0, 68.5)
- added R5: 220 Ohm, Resistor_THT:R_Axial_DIN0204_L3.6mm_D1.6mm_P5.08mm_Vertical, F.Cu at (181.0, 68.5)
- added R6: 220 Ohm, Resistor_THT:R_Axial_DIN0204_L3.6mm_D1.6mm_P5.08mm_Vertical, F.Cu at (178.0, 68.5)
- added U1: 74HC595, Package_SO:SO-16_3.9x9.9mm_P1.27mm, F.Cu at (172.4, 102.4)
- added U2: 74HC165, Package_SO:SO-16_3.9x9.9mm_P1.27mm, F.Cu at (172.4, 116.4)
- moved H1 1.48 mm to (95.0, 86.0)
- moved H2 1.17 mm to (120.0, 86.0)
- moved H4 0.83 mm to (120.0, 136.0)
- moved H3 0.78 mm to (95.0, 136.0)
Routing:
- net Net-(A1-+5V): track 0.00 -> 123.2 mm
- net Net-(A1-A0): track 0.00 -> 66.1 mm
- net Net-(J10-Pin_2): track 0.00 -> 64.1 mm
- net Net-(A1-A1): track 0.00 -> 52.4 mm
- net Net-(A1-D10): track 0.00 -> 50.7 mm
- net Net-(U1-QC): track 0.00 -> 46.0 mm
- net Net-(U1-QB): track 0.00 -> 45.4 mm
- net Net-(A1-D9): track 0.00 -> 45.3 mm
- net Net-(U1-QD): track 0.00 -> 44.7 mm
- net Net-(U1-QA): track 0.00 -> 43.7 mm
- net Net-(U1-QE): track 0.00 -> 43.7 mm
- net Net-(U1-QF): track 0.00 -> 43.3 mm
- net Net-(A1-D8): track 0.00 -> 39.9 mm
- net Net-(A1-A2): track 0.00 -> 38.2 mm, vias 0 -> 1
- net Net-(A1-D7): track 0.00 -> 34.6 mm
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Other:
- board outline added: 37 x 62 mm
- board text added: "v .1 CountCounter Daugter Board"
